File: PCB/PCB.kicad_sch (KiCad schematic)
At the start: 0 parts

Commit message: a
Parts:
- added C1, C11, C12, C2, C3, C4, C5, C6, C7, C8: 0.1uF, symbol Device:C
- added C10, C9: 1uF, symbol Device:C
- added C13, C14: 10uF, symbol Device:C
- added J2: USB_C_Receptacle_USB2.0_14P, symbol Connector:USB_C_Receptacle_USB2.0_14P
- added R1, R2: 5.1K, symbol Device:R
- added R3, R4: 27, symbol Device:R
- added U1: RP2040, Package_DFN_QFN:QFN-56-1EP_7x7mm_P0.4mm_EP3.2x3.2mm, symbol MCU_RaspberryPi:RP2040
- added U2: NCP1117-3.3_SOT223, Package_TO_SOT_SMD:SOT-223-3_TabPin2, symbol Regulator_Linear:NCP1117-3.3_SOT223
- added Y1: Crystal_GND24, symbol Device:Crystal_GND24
Connections:
- new net: R4.2, U1.46 (USB_DM)
- new net: J2.B5 (CC2), R2.1
- new net: R3.2, U1.47 (USB_DP)
- new net: J2.A5 (CC1), R1.1
- new net +1V1: C10.1, C11.1, C12.1, U1.23 (DVDD), U1.45 (VREG_VOUT), U1.50 (DVDD)
- new net +3V3: C1.1, C14.1, C2.1, C3.1, C4.1, C5.1, C6.1, C7.1, C8.1, C9.1, U1.1 (IOVDD), U1.10 (IOVDD), U1.22 (IOVDD), U1.33 (IOVDD), U1.42 (IOVDD), U1.43 (ADC_AVDD), U1.44 (VREG_IN), U1.48 (USB_VDD), U1.49 (IOVDD), U2.2 (VO)
- new net GND: C1.2, C10.2, C11.2, C12.2, C13.2, C14.2, C2.2, C3.2, C4.2, C5.2, C6.2, C7.2, C8.2, C9.2, J2.A1 (GND), J2.A12 (GND), J2.B1 (GND), J2.B12 (GND), J2.S1 (SHIELD), R1.2, R2.2, U1.57 (GND), U2.1 (GND)
- new net USBD+: J2.A6 (D+), J2.B6 (D+), R3.1
- new net USBD-: J2.A7 (D-), J2.B7 (D-), R4.1
- new net VBUS: C13.1, J2.A4 (VBUS), J2.A9 (VBUS), J2.B4 (VBUS), J2.B9 (VBUS), U2.3 (VI)
- new net XIN: U1.20 (XIN)
- new net XOUT: U1.21 (XOUT)
